File: LED_PCB/LED_PCB.sch (KiCad schematic (older format))
At the start: 62 parts

Commit message: Finished schematic & BOM, started layout, need to define PCB shape
Parts:
- removed C? (x17): C_Small, symbol C_Small
- removed D? (x7): LED_THERMAL_PAD, symbol LED_THERMAL_PAD
- removed J? (x5): TEST_1P, symbol TEST_1P
- removed R? (x9): R_Small, symbol R_Small
- added C10, C11, C12, C13, C14, C15, C16, C17, C18, C2, C4, C7, C8, C9: 0.1uF, Capacitors_SMD:C_0603_HandSoldering, symbol C_Small
- added C3, C5, C6: 4.7uF, Capacitors_SMD:C_0805_HandSoldering, symbol C_Small
- added D2, D3, D4, D5, D6, D7, D8: XMLBWT-x, buq2:CREE-XM-L, symbol LED_THERMAL_PAD
- added J11, J12, J13, J3, J5, J6, J7, J8, J9: TEST_1P, SMD_Packages:1Pin, symbol TEST_1P
- added R1, R11, R2, R7, R8, R9: 1k, Resistors_SMD:R_0603_HandSoldering, symbol R_Small
- added R10, R5: 0 OHM, Resistors_SMD:R_0603_HandSoldering, symbol R_Small
- added R3: 10k, Resistors_SMD:R_0603_HandSoldering, symbol R_Small
- C1: renamed from C?; value C_Small -> 4.7uF; footprint (none) -> Capacitors_SMD:C_0805_HandSoldering
- D1: renamed from D?; value LED_THERMAL_PAD -> XMLBWT-x; footprint (none) -> buq2:CREE-XM-L
- J1, J2, J4: renamed from J?; footprint (none) -> Connectors:1pin
- J10: renamed from J?; footprint (none) -> SMD_Packages:1Pin
- Q1: renamed from Q?; footprint (none) -> TO_SOT_Packages_SMD:SOT-23
- Q2: renamed from Q?; footprint (none) -> TO_SOT_Packages_SMD:TO-252-2_Rectifier
- R4: renamed from R?; value R_Small -> 10k; footprint (none) -> Resistors_SMD:R_0603_HandSoldering
- R6: renamed from R?; value R_Small -> 1k; footprint (none) -> Resistors_SMD:R_0603_HandSoldering
- gave numbers to parts that had none: 14
Connections:
- net +3V3: now also C2.1, C5.1, J6.1
- net DOUT: now also J11.1, R7.2
- net GND: now also C10.2, C11.2, C12.2, C13.2, C14.2, C15.2, C16.2, C17.2, C18.2, C2.2, C3.2, C4.2, C5.2, C6.2, C7.2, C8.2, C9.2, D8.1 (K), J3.1, R2.2, R3.2
- net MODE: now also J12.1, R3.1, R8.2
- net VDD: now also C10.1, C11.1, C12.1, C13.1, C14.1, C15.1, C16.1, C17.1, C18.1, C6.1, C7.1, C8.1, C9.1, J7.1
- net VIN_ADC: now also C4.1, J13.1, R1.2, R10.2, R2.1
- net at U2.1 (PB5(~RESET~/dW/ADC0/PCINT5)): now also R11.1
- net at U2.2 (PB3(XTAL1/CLKI/~OC1B~/ADC3/PCINT3)): now also R9.1
- net at U2.3 (PB4(XTAL2/CLKO/OC1B/ADC2/PCINT4)): now also R10.1
- net at U2.6 (PB1(MISO/DO/AIN1/OC0B/OC1A/PCINT1)): now also R7.1
- net at U2.7 (PB2(SCK/USCK/SCL/T0/INT0/ADC1/PCINT2)): now also R8.1
- net at Q2.1 (G), R4.2: now also R5.1
- net at C1.1, D1.2 (A), J1.1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: now also C3.1, J5.1, R1.1
- net at Q1.3 (D): now also R5.2
- net at LED8.2 (DOUT): now also LED9.4 (DIN)
- net at D1.1 (K): now also D2.2 (A)
- new net: D2.1 (K), D3.2 (A)
- new net: D3.1 (K), D4.2 (A)
- new net: D4.1 (K), D5.2 (A)
- new net: D5.1 (K), D6.2 (A)
- new net: D6.1 (K), D7.2 (A)
- new net: D7.1 (K), D8.2 (A)
- new net: J8.1, R9.2
- new net: J9.1, R11.2

Commit message: LED board: routed most of top layer... started controller PCB schematic.
Parts:
- removed J9: TEST_1P, SMD_Packages:1Pin, symbol TEST_1P
- added C19: 1000pF, Capacitors_SMD:C_0603_HandSoldering, symbol C_Small
- added J9: Conn_01x06, Pin_Headers:Pin_Header_Straight_1x06_Pitch2.54mm_SMD_Pin1Left, symbol Conn_01x06
- added R12: 0 OHM, Resistors_SMD:R_0603_HandSoldering, symbol R_Small
- J10, J11, J12, J13, J3, J5, J6, J7, J8: footprint SMD_Packages:1Pin -> Measurement_Points:Measurement_Point_Round-SMD-Pad_Small
- R11: value 1k -> 10k
Connections:
- net +3V3 is gone; now on net VCC: C2.1, C5.1, J6.1, U1.2 (OUT), U1.4 (VOUT), U2.8 (VCC)
- net GND: now also C19.1, J9.2 (Pin_2)
- net at R11.1, U2.1 (PB5(~RESET~/dW/ADC0/PCINT5)): now also C19.2, J9.6 (Pin_6)
- net at R6.1, U2.5 (PB0(MOSI/DI/SDA/AIN0/OC0A/~OC1A~/AREF/PCINT0)): now also J9.5 (Pin_5)
- net at R7.1, U2.6 (PB1(MISO/DO/AIN1/OC0B/OC1A/PCINT1)): now also J9.4 (Pin_4)
- net at R8.1, U2.7 (PB2(SCK/USCK/SCL/T0/INT0/ADC1/PCINT2)): now also J9.3 (Pin_3)
- net at C1.1, C3.1, D1.2 (A)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: now also R12.1
- net VCC: now reaches R11.2
- net VCC: now also J9.1 (Pin_1), R12.2

Commit message: Added components to LED PCB sch and updated layout
Still need to add thermals for white LEDs and then run error check...
Parts:
- removed U1: AZ1117CH-3_3TRG1, digikey-footprints:SOT-223, symbol AZ1117CH-3_3TRG1
- added D9: BAT54S-7-F, digikey-footprints:SOT-23-3, symbol BAT54S-7-F
- added Q3: Q_NMOS_SDG, TO_SOT_Packages_SMD:SOT-89-3_Handsoldering, symbol Q_NMOS_SDG
- added R13: 0 OHM, Resistors_SMD:R_0603_HandSoldering, symbol R_Small
- added R14: 10k, Resistors_SMD:R_0603_HandSoldering, symbol R_Small
- added U1: MIC5233-3.3YS-TR, TO_SOT_Packages_SMD:SOT-223, symbol MIC5233-3.3YS-TR
- D1, D2, D3, D4, D5, D6, D7, D8: footprint buq2:CREE-XM-L -> CustomFootprints:CREE-XM-L_HAND_SOLDERED
Connections:
- net GND: now also D1.3 (PAD), D2.3 (PAD), D3.3 (PAD), D4.3 (PAD), D5.3 (PAD), D6.3 (PAD), D7.3 (PAD), D8.3 (PAD), D9.1, Q3.1 (S), R14.2, U1.2 (GND), U1.4 (GND); no longer D8.1 (K)
- net VCC: now also D9.2, U1.3 (OUT)
- net VIN_ADC: now also D9.3
- net at C1.1, C3.1, J1.1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: now also R13.2, U1.1 (IN); no longer D1.2 (A)
- net WHITE_EN: now reaches J8.1, R9.2
- net WHITE_EN: now also Q3.3 (G), R14.1
- net MODE renamed RGB_EN
- new net: D1.2 (A), R13.1
- new net: D8.1 (K), Q3.2 (D)
- no-connect marks 0 -> 1
Other:
- note added: "Init: RGB_EN and WHITE_EN low... read VIN\nVIN <= 5.3V: Use RGB LEDs -> RGB_EN high, WHITE_EN low\nVIN > 6V: Upstream converter driving white LEDs, WHITE_EN high, RGB_EN low"
- moved on the sheet: J8
