File: POWER_PCB/Input_Output.sch (KiCad schematic (older format))
At the start: 36 parts

Commit message: Updated POWER_PCB & CONTROLLER_PCB sch's and layouts
Parts:
- removed C?: 10uF, Capacitors_SMD:C_0805_HandSoldering, symbol C_Small
- removed C?: 0.01uF, Capacitors_SMD:C_0603_HandSoldering, symbol C_Small
- removed FL?: EMI_Filter_LL, CustomFootprints:IND_ACM12V-701-2PL-TL00_FixedPadNumbers, symbol EMI_Filter_LL
- removed R?: 2.49k, Resistors_SMD:R_0603_HandSoldering, symbol R_Small
- removed R?: 10k, Resistors_SMD:R_0603_HandSoldering, symbol R_Small
- added C20, C21, C8: 22uF, Capacitors_SMD:C_1206_HandSoldering, symbol C_Small
- added F1: Polyfuse, 2920L:2920L, symbol Polyfuse
- added FL1: EMI_Filter_LL_14_23, ACM70V-701-2PL-TL00:FIL_ACM70V-701-2PL-TL00, symbol EMI_Filter_LL_14_23
- added TP7, TP8, TP9: TEST, Measurement_Points:Measurement_Point_Round-SMD-Pad_Small, symbol TEST
- J3, J4, J5, J6: renamed from J?; footprint (none) -> Pin_Headers:Pin_Header_Straight_1x02_Pitch2.54mm
- L1: renamed from L?; footprint CustomFootprints:L_12x12mm_h8mm_hand_soldering -> Inductors_SMD:L_Vishay_IHLP-1616
- gave numbers to parts that had none: 26
Connections:
- net BOOST_BYPASS: now also TP8.1
- net BOOST_EN: now also TP9.1
- net GND: now also C20.2, C21.2, C8.2, FL1.3
- net Vin: now also C7.1, C20.1
- net Vout: now also C21.1, TP7.1
- net at C1.2, C2.2, C3.2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: now also FL1.2
- net at C4.1, C5.1, D1.2 (K)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: now also FL1.1
- new net: C8.1, F1.1, L1.1
- new net: C6.1, F1.2, FL1.4
Other:
- moved on the sheet: C6, C7, L1, TP2
