File: POWER_PCB/LED_Boost.sch (KiCad schematic (older format))
At the start: 25 parts

Commit message: Updated POWER_PCB & CONTROLLER_PCB sch's and layouts
Parts:
- removed TP? (x2): TEST, Measurement_Points:Measurement_Point_Round-SMD-Pad_Small, symbol TEST
- added C18, C19: 10uF, Capacitors_SMD:C_0805_HandSoldering, symbol C_Small
- added J10: Conn_01x02, Pin_Headers:Pin_Header_Straight_1x02_Pitch2.54mm, symbol Conn_01x02
- added TP10: TEST, Measurement_Points:Measurement_Point_Round-SMD-Pad_Small, symbol TEST
- L2: renamed from L?; footprint CustomFootprints:L_12x12mm_h8mm_hand_soldering -> Inductors_SMD:L_Vishay_IHLP-2525
- gave numbers to parts that had none: 21
Connections:
- net BOOST_OUT: now also C19.1
- net GND: now also C18.2, C19.2
- net LED_RTN: now also TP10.1
- net Vin: now also C18.1
- net at R15.1, U2.9 (FB): now also J10.1 (Pin_1)
- net at R13.1, R15.2, U1.1: now also J10.2 (Pin_2)
Other:
- moved on the sheet: C9
